File: power-distribution-board/power-distribution-board.kicad_pcb (KiCad board)
At the start: 2 copper layers, 90 x 70 mm, 23 parts, among them J1 Conn_01x02, J2 Conn_01x02, J3 Conn_01x02, J4 Conn_01x02, J5 Conn_01x02, J6 Conn_01x02, J7 Conn_01x02, J8 Conn_01x02

Commit message: 完成
Parts:
- added G***: LOGO, LOGO, F.Cu at (100.3, 55.0)
- moved D1 3.40 mm to (42.0, 16.0)
- moved R1 3.40 mm to (45.4, 16.0)
Connections:
- D1 pad 1: Net-(D1-K) -> GND
- D1 pad 2: VCC -> Net-(D1-A)
- R1 pad 1: Net-(D1-K) -> VCC
- R1 pad 2: GND -> Net-(D1-A)
Routing:
- net Net-(D1-K): track 1.61 -> 0.00 mm
- net Net-(D1-A): track 0.00 -> 1.57 mm
- net VCC: vias 0 -> 106
- net GND: vias 0 -> 110
Other:
- board text added: "GND"
- board text added: "power-distribution-board version 1.0 create by ikeda"
